File: gaming-clock/gaming-clock.kicad_pcb (KiCad board)
At the start: 2 copper layers, 207.5 x 67.6 mm, 2 parts

Commit message: led
Parts:
- removed REF**: LED_SK6812MINI_PLCC4_3.5x3.5mm_P1.75mm, LED_SMD:LED_SK6812MINI_PLCC4_3.5x3.5mm_P1.75mm
- removed REF**: ESP32-C3-WROOM-02, Espressif:ESP32-C3-WROOM-02
Changed lines of the file:
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@@
   )
   (net 0 "")
-  (footprint "LED_SMD:LED_SK6812MINI_PLCC4_3.5x3.5mm_P1.75mm" (layer "F.Cu")
-    (at 126.492 93.98)
-    (descr "https://cdn-shop.adafruit.com/product-files/2686/SK6812MINI_REV.01-1-2.pdf")
-    (tags "LED RGB NeoPixel Mini")
-    (attr smd)
-    (fp_text reference "REF**" (at 0 -2.75) (layer "F.SilkS")
-        (effects (font (size 1 1) (thickness 0.15)))
-    )
-    (fp_text value "LED_SK6812MINI_PLCC4_3.5x3.5mm_P1.75mm" (at 0 3.25) (layer "F.Fab")
-        (effects (font (size 1 1) (thickness 0.15)))
-    )
-    (fp_text user "1" (at -3.5 -0.875) (layer "F.SilkS")
-        (effects (font (size 1 1) (thickness 0.15)))
-    )
-    (fp_text user "${REFERENCE}" (at 0 0) (layer "F.Fab")
-        (effects (font (size 0.5 0.5) (thickness 0.1)))
-    )
-    (fp_line (start -2.95 -1.95) (end 2.95 -1.95)
-      (stroke (width 0.12) (type solid)) (layer "F.SilkS"))
-    (fp_line (start -2.95 1.95) (end 2.95 1.95)
-      (stroke (width 0.12) (type solid)) (layer "F.SilkS"))
-    (fp_line (start 2.95 1.95) (end 2.95 0.875)
-      (stroke (width 0.12) (type solid)) (layer "F.SilkS"))
-    (fp_line (start -2.8 -2) (end -2.8 2)
-      (stroke (width 0.05) (type solid)) (layer "F.CrtYd"))
-    (fp_line (start -2.8 2) (end 2.8 2)
-      (stroke (width 0.05) (type solid)) (layer "F.CrtYd"))
-    (fp_line (start 2.8 -2) (end -2.8 -2)
-      (stroke (width 0.05) (type solid)) (layer "F.CrtYd"))
-    (fp_line (start 2.8 2) (end 2.8 -2)
-      (stroke (width 0.05) (type solid)) (layer "F.CrtYd"))
-    (fp_line (start -1.75 -1.75) (end -1.75 1.75)
-      (stroke (width 0.1) (type solid)) (layer "F.Fab"))
-    (fp_line (start -1.75 1.75) (end 1.75 1.75)
-      (stroke (width 0.1) (type solid)) (layer "F.Fab"))
-    (fp_line (start 1.75 -1.75) (end -1.75 -1.75)
-      (stroke (width 0.1) (type solid)) (layer "F.Fab"))
-    (fp_line (start 1.75 0.75) (end 0.75 1.75)
-      (stroke (width 0.1) (type solid)) (layer "F.Fab"))
-    (fp_line (start 1.75 1.75) (end 1.75 -1.75)
-      (stroke (width 0.1) (type solid)) (layer "F.Fab"))
-    (fp_circle (center 0 0) (end 0 -1.5)
-      (stroke (width 0.1) (type solid)) (fill none) (layer "F.Fab"))
-    (pad "1" smd rect (at -1.75 -0.875) (size 1.6 0.85) (layers "F.Cu" "F.Paste" "F.Mask"))
-    (pad "2" smd rect (at -1.75 0.875) (size 1.6 0.85) (layers "F.Cu" "F.Paste" "F.Mask"))
-    (pad "3" smd rect (at 1.75 0.875) (size 1.6 0.85) (layers "F.Cu" "F.Paste" "F.Mask"))
-    (pad "4" smd rect (at 1.75 -0.875) (size 1.6 0.85) (layers "F.Cu" "F.Paste" "F.Mask"))
-    (model ":KICAD7_3DMODEL_DIR:LED_SMD.3dshapes/LED_SK6812_PLCC4_5.0x5.0mm_P3.2mm.step"
-      (offset (xyz 0 0 0))
-      (scale (xyz 1 1 1))
-      (rotate (xyz 0 0 0))
-    )
-  )
-  (footprint "Espressif:ESP32-C3-WROOM-02" (layer "B.Cu")
-    (at 179.88 81.026 90)
-    (descr "ESP32-C3-WROOM-02: https://www.espressif.com/sites/default/files/documentation/esp32-c3-wroom-02_datasheet_en.pdf")
-    (tags "ESP32-C3")
-    (attr smd)
-    (fp_text reference "REF**" (at 0 14.75 90) (layer "B.SilkS")
-        (effects (font (size 1 1) (thickness 0.15)) (justify mirror))
-    )
-    (fp_text value "ESP32-C3-WROOM-02" (at 0 -8.75 90) (layer "B.Fab")
-        (effects (font (size 1 1) (thickness 0.15)) (justify mirror))
-    )
-    (fp_text user "Antenna Area" (at 0 10.4 90) (layer "B.SilkS")
-        (effects (font (size 1 1) (thickness 0.15)) (justify mirror))
-    )
-    (fp_text user "${REFERENCE}" (at 0 1.75 90) (layer "B.Fab")
-        (effects (font (size 1 1) (thickness 0.15)) (justify mirror))
-    )
-    (fp_line (start -9 -7) (end -9 -6.75)
-      (stroke (width 0.12) (type solid)) (layer "B.SilkS"))
-    (fp_line (start -9 13) (end -9 6.5)
-      (stroke (width 0.12) (type solid)) (layer "B.SilkS"))
-    (fp_line (start -9 13) (end 9 13)
-      (stroke (width 0.12) (type solid)) (layer "B.SilkS"))
-    (fp_line (start 9 -7) (end -9 -7)
-      (stroke (width 0.12) (type solid)) (layer "B.SilkS"))
-    (fp_line (start 9 -6.75) (end 9 -7)
-      (stroke (width 0.12) (type solid)) (layer "B.SilkS"))
-    (fp_line (start 9 7) (end -8.95 7)
-      (stroke (width 0.12) (type solid)) (layer "B.SilkS"))
-    (fp_line (start 9 13) (end 9 6.5)
-      (stroke (width 0.12) (type solid)) (layer "B.SilkS"))
-    (fp_poly
-      (pts
-        (xy 9.8 -7.3)
-        (xy -9.8 -7.3)
-        (xy -9.8 13.3)
-        (xy 9.8 13.3)
-      )
-      (stroke (width 0.05) (type solid)) (fill none) (layer "B.CrtYd"))
-    (fp_line (start -9 -7) (end -9 13)
-      (stroke (width 0.1) (type solid)) (layer "B.Fab"))
-    (fp_line (start -9 7) (end 9 7)
-      (stroke (width 0.1) (type solid)) (layer "B.Fab"))
-    (fp_line (start -9 13) (end 9 13)
-      (stroke (width 0.1) (type solid)) (layer "B.Fab"))
-    (fp_line (start -7.7 7) (end -9 5.7)
-      (stroke (width 0.1) (type solid)) (layer "B.Fab"))
-    (fp_line (start 9 -7) (end -9 -7)
-      (stroke (width 0.1) (type solid)) (layer "B.Fab"))
-    (fp_line (start 9 13) (end 9 -7)
-      (stroke (width 0.1) (type solid)) (layer "B.Fab"))
-    (pad "1" smd rect (at -8.75 5.9 90) (size 1.5 0.9) (layers "B.Cu" "B.Paste" "B.Mask"))
-    (pad "2" smd rect (at -8.75 4.4 90) (size 1.5 0.9) (layers "B.Cu" "B.Paste" "B.Mask"))
-    (pad "3" smd rect (at -8.75 2.9 90) (size 1.5 0.9) (layers "B.Cu" "B.Paste" "B.Mask"))
-    (pad "4" smd rect (at -8.75 1.4 90) (size 1.5 0.9) (layers "B.Cu" "B.Paste" "B.Mask"))
-    (pad "5" smd rect (at -8.75 -0.1 90) (size 1.5 0.9) (layers "B.Cu" "B.Paste" "B.Mask"))
-    (pad "6" smd rect (at -8.75 -1.6 90) (size 1.5 0.9) (layers "B.Cu" "B.Paste" "B.Mask"))
-    (pad "7" smd rect (at -8.75 -3.1 90) (size 1.5 0.9) (layers "B.Cu" "B.Paste" "B.Mask"))
-    (pad "8" smd rect (at -8.75 -4.6 90) (size 1.5 0.9) (layers "B.Cu" "B.Paste" "B.Mask"))
-    (pad "9" smd rect (at -8.75 -6.1 90) (size 1.5 0.9) (layers "B.Cu" "B.Paste" "B.Mask"))
-    (pad "10" smd rect (at 8.75 -6.1 270) (size 1.5 0.9) (layers "B.Cu" "B.Paste" "B.Mask"))
-    (pad "11" smd rect (at 8.75 -4.6 270) (size 1.5 0.9) (layers "B.Cu" "B.Paste" "B.Mask"))
-    (pad "12" smd rect (at 8.75 -3.1 270) (size 1.5 0.9) (layers "B.Cu" "B.Paste" "B.Mask"))
-    (pad "13" smd rect (at 8.75 -1.6 270) (size 1.5 0.9) (layers "B.Cu" "B.Paste" "B.Mask"))
-    (pad "14" smd rect (at 8.75 -0.1 270) (size 1.5 0.9) (layers "B.Cu" "B.Paste" "B.Mask"))
-    (pad "15" smd rect (at 8.75 1.4 270) (size 1.5 0.9) (layers "B.Cu" "B.Paste" "B.Mask"))
-    (pad "16" smd rect (at 8.75 2.9 270) (size 1.5 0.9) (layers "B.Cu" "B.Paste" "B.Mask"))
-    (pad "17" smd rect (at 8.75 4.4 270) (size 1.5 0.9) (layers "B.Cu" "B.Paste" "B.Mask"))
-    (pad "18" smd rect (at 8.75 5.9 270) (size 1.5 0.9) (layers "B.Cu" "B.Paste" "B.Mask"))
-    (pad "19" smd rect (at -0.14 -1.4 270) (size 0.7 0.7) (layers "B.Cu" "B.Paste" "B.Mask"))
-    (pad "19" smd rect (at -0.14 -0.3 270) (size 0.7 0.7) (layers "B.Cu" "B.Paste" "B.Mask"))
-    (pad "19" smd rect (at -0.14 0.8 270) (size 0.7 0.7) (layers "B.Cu" "B.Paste" "B.Mask"))
-    (pad "19" smd rect (at 0.91 -1.4 270) (size 0.7 0.7) (layers "B.Cu" "B.Paste" "B.Mask"))
-    (pad "19" smd rect (at 0.91 -0.3 270) (size 0.7 0.7) (layers "B.Cu" "B.Paste" "B.Mask"))
-    (pad "19" smd rect (at 0.91 0.8 270) (size 0.7 0.7) (layers "B.Cu" "B.Paste" "B.Mask"))
-    (pad "19" smd rect (at 2.06 -1.4 270) (size 0.7 0.7) (layers "B.Cu" "B.Paste" "B.Mask"))
-    (pad "19" smd rect (at 2.06 -0.3 270) (size 0.7 0.7) (layers "B.Cu" "B.Paste" "B.Mask"))
-    (pad "19" smd rect (at 2.06 0.8 270) (size 0.7 0.7) (layers "B.Cu" "B.Paste" "B.Mask"))
-    (zone (net 0) (net_name "") (layers "*.Cu") (name "antenna keepout") (hatch edge 0.508)
-      (connect_pads (clearance 0))
-      (min_thickness 0.254) (filled_areas_thickness no)
-      (keepout (tracks not_allowed) (vias not_allowed) (pads not_allowed) (copperpour not_allowed) (footprints not_allowed))
-      (fill (thermal_gap 0.508) (thermal_bridge_width 0.508))
-      (polygon
-        (pts
-          (xy 186.88 72.026)
-          (xy 186.88 90.026)
-          (xy 192.88 90.026)
-          (xy 192.88 72.026)
-        )
-      )
-    )
-    (model "${KIPRJMOD}/library/3dmodels/espressif.3dshapes/ESP32-C3-WROOM-02.STEP"
-      (offset (xyz -9 -7 0))
-      (scale (xyz 1 1 1))
-      (rotate (xyz 0 0 0))
-    )
-  )
   (gr_line (start 121.412 89.662) (end 144.272 89.662)
     (stroke (width 0.1) (type default)) (layer "Edge.Cuts"))

Commit message: fin
Parts:
- added C1: 10u, Capacitor_SMD:C_0603_1608Metric_Pad1.08x0.95mm_HandSolder, F.Cu at (182.2, 102.4)
- added C10: 10u, Capacitor_SMD:C_0603_1608Metric_Pad1.08x0.95mm_HandSolder, F.Cu at (175.6, 111.1)
- added C2: 100n, Capacitor_SMD:C_0603_1608Metric_Pad1.08x0.95mm_HandSolder, F.Cu at (182.2, 100.8)
- added C201: 10u, Capacitor_SMD:C_0603_1608Metric_Pad1.08x0.95mm_HandSolder, F.Cu at (271.2, 78.0)
- added C202: 10u, Capacitor_SMD:C_0603_1608Metric_Pad1.08x0.95mm_HandSolder, F.Cu at (271.0, 109.2)
- added C203: 10u, Capacitor_SMD:C_0603_1608Metric_Pad1.08x0.95mm_HandSolder, F.Cu at (256.5, 93.7)
- added C204: 10u, Capacitor_SMD:C_0603_1608Metric_Pad1.08x0.95mm_HandSolder, F.Cu at (256.5, 63.5)
- added C205: 10u, Capacitor_SMD:C_0603_1608Metric_Pad1.08x0.95mm_HandSolder, F.Cu at (256.3, 123.9)
- added C206: 10u, Capacitor_SMD:C_0603_1608Metric_Pad1.08x0.95mm_HandSolder, F.Cu at (241.5, 78.2)
- added C207: 10u, Capacitor_SMD:C_0603_1608Metric_Pad1.08x0.95mm_HandSolder, F.Cu at (241.5, 109.0)
- added C3: 100n, Capacitor_SMD:C_0603_1608Metric_Pad1.08x0.95mm_HandSolder, F.Cu at (185.4, 91.9)
- added C301: 10u, Capacitor_SMD:C_0603_1608Metric_Pad1.08x0.95mm_HandSolder, F.Cu at (223.8, 78.0)
- added C302: 10u, Capacitor_SMD:C_0603_1608Metric_Pad1.08x0.95mm_HandSolder, F.Cu at (223.5, 109.2)
- added C303: 10u, Capacitor_SMD:C_0603_1608Metric_Pad1.08x0.95mm_HandSolder, F.Cu at (209.1, 93.7)
- added C304: 10u, Capacitor_SMD:C_0603_1608Metric_Pad1.08x0.95mm_HandSolder, F.Cu at (209.1, 63.5)
- added C305: 10u, Capacitor_SMD:C_0603_1608Metric_Pad1.08x0.95mm_HandSolder, F.Cu at (208.8, 124.0)
- added C306: 10u, Capacitor_SMD:C_0603_1608Metric_Pad1.08x0.95mm_HandSolder, F.Cu at (194.1, 78.2)
- added C307: 10u, Capacitor_SMD:C_0603_1608Metric_Pad1.08x0.95mm_HandSolder, F.Cu at (194.1, 109.0)
- added C4: 10u, Capacitor_SMD:C_0603_1608Metric_Pad1.08x0.95mm_HandSolder, F.Cu at (180.5, 91.9)
- added C401: 10u, Capacitor_SMD:C_0603_1608Metric_Pad1.08x0.95mm_HandSolder, F.Cu at (117.9, 109.5)
- added C402: 10u, Capacitor_SMD:C_0603_1608Metric_Pad1.08x0.95mm_HandSolder, F.Cu at (118.1, 78.2)
- added C403: 10u, Capacitor_SMD:C_0603_1608Metric_Pad1.08x0.95mm_HandSolder, F.Cu at (132.6, 93.7)
- added C404: 10u, Capacitor_SMD:C_0603_1608Metric_Pad1.08x0.95mm_HandSolder, F.Cu at (132.6, 124.0)
- added C405: 10u, Capacitor_SMD:C_0603_1608Metric_Pad1.08x0.95mm_HandSolder, F.Cu at (132.8, 63.5)
- added C406: 10u, Capacitor_SMD:C_0603_1608Metric_Pad1.08x0.95mm_HandSolder, F.Cu at (147.6, 109.2)
- added C407: 10u, Capacitor_SMD:C_0603_1608Metric_Pad1.08x0.95mm_HandSolder, F.Cu at (147.6, 78.5)
- added C501: 10u, Capacitor_SMD:C_0603_1608Metric_Pad1.08x0.95mm_HandSolder, F.Cu at (70.4, 109.5)
- added C502: 10u, Capacitor_SMD:C_0603_1608Metric_Pad1.08x0.95mm_HandSolder, F.Cu at (70.6, 78.3)
- added C503: 10u, Capacitor_SMD:C_0603_1608Metric_Pad1.08x0.95mm_HandSolder, F.Cu at (85.1, 93.8)
- added C504: 10u, Capacitor_SMD:C_0603_1608Metric_Pad1.08x0.95mm_HandSolder, F.Cu at (85.1, 124.0)
- added C505: 10u, Capacitor_SMD:C_0603_1608Metric_Pad1.08x0.95mm_HandSolder, F.Cu at (85.3, 63.5)
- added C506: 10u, Capacitor_SMD:C_0603_1608Metric_Pad1.08x0.95mm_HandSolder, F.Cu at (100.1, 109.2)
- added C507: 10u, Capacitor_SMD:C_0603_1608Metric_Pad1.08x0.95mm_HandSolder, F.Cu at (100.1, 78.5)
- added C7: 10u, Capacitor_SMD:C_0603_1608Metric_Pad1.08x0.95mm_HandSolder, F.Cu at (169.5, 74.3)
- added C8: 10u, Capacitor_SMD:C_0603_1608Metric_Pad1.08x0.95mm_HandSolder, F.Cu at (167.0, 85.7)
- added C9: 10u, Capacitor_SMD:C_0603_1608Metric_Pad1.08x0.95mm_HandSolder, F.Cu at (175.6, 101.6)
- added D1: SK6812MINI, LED_SMD:LED_SK6812MINI_PLCC4_3.5x3.5mm_P1.75mm, F.Cu at (162.6, 78.4)
- added D2: SK6812MINI, LED_SMD:LED_SK6812MINI_PLCC4_3.5x3.5mm_P1.75mm, F.Cu at (179.1, 78.4)
- added D201: SK6812MINI, LED_SMD:LED_SK6812MINI_PLCC4_3.5x3.5mm_P1.75mm, F.Cu at (271.1, 115.4)
- added D202: SK6812MINI, LED_SMD:LED_SK6812MINI_PLCC4_3.5x3.5mm_P1.75mm, F.Cu at (271.1, 103.0)
- added D203: SK6812MINI, LED_SMD:LED_SK6812MINI_PLCC4_3.5x3.5mm_P1.75mm, F.Cu at (271.1, 84.4)
- added D204: SK6812MINI, LED_SMD:LED_SK6812MINI_PLCC4_3.5x3.5mm_P1.75mm, F.Cu at (271.1, 72.0)
- added D205: SK6812MINI, LED_SMD:LED_SK6812MINI_PLCC4_3.5x3.5mm_P1.75mm, F.Cu at (262.5, 124.1)
- added D206: SK6812MINI, LED_SMD:LED_SK6812MINI_PLCC4_3.5x3.5mm_P1.75mm, F.Cu at (262.5, 93.7)
- added D207: SK6812MINI, LED_SMD:LED_SK6812MINI_PLCC4_3.5x3.5mm_P1.75mm, F.Cu at (262.5, 63.4)
- added D208: SK6812MINI, LED_SMD:LED_SK6812MINI_PLCC4_3.5x3.5mm_P1.75mm, F.Cu at (250.0, 124.1)
- added D209: SK6812MINI, LED_SMD:LED_SK6812MINI_PLCC4_3.5x3.5mm_P1.75mm, F.Cu at (250.0, 93.7)
- added D210: SK6812MINI, LED_SMD:LED_SK6812MINI_PLCC4_3.5x3.5mm_P1.75mm, F.Cu at (250.0, 63.4)
- added D211: SK6812MINI, LED_SMD:LED_SK6812MINI_PLCC4_3.5x3.5mm_P1.75mm, F.Cu at (241.4, 115.4)
- added D212: SK6812MINI, LED_SMD:LED_SK6812MINI_PLCC4_3.5x3.5mm_P1.75mm, F.Cu at (241.4, 103.0)
- added D213: SK6812MINI, LED_SMD:LED_SK6812MINI_PLCC4_3.5x3.5mm_P1.75mm, F.Cu at (241.4, 84.4)
- added D214: SK6812MINI, LED_SMD:LED_SK6812MINI_PLCC4_3.5x3.5mm_P1.75mm, F.Cu at (241.4, 72.0)
- added D3: SK6812MINI, LED_SMD:LED_SK6812MINI_PLCC4_3.5x3.5mm_P1.75mm, F.Cu at (170.8, 85.6)
- added D301: SK6812MINI, LED_SMD:LED_SK6812MINI_PLCC4_3.5x3.5mm_P1.75mm, F.Cu at (223.7, 115.4)
- added D302: SK6812MINI, LED_SMD:LED_SK6812MINI_PLCC4_3.5x3.5mm_P1.75mm, F.Cu at (223.7, 103.0)
- added D303: SK6812MINI, LED_SMD:LED_SK6812MINI_PLCC4_3.5x3.5mm_P1.75mm, F.Cu at (223.7, 84.5)
- added D304: SK6812MINI, LED_SMD:LED_SK6812MINI_PLCC4_3.5x3.5mm_P1.75mm, F.Cu at (223.7, 72.0)
- added D305: SK6812MINI, LED_SMD:LED_SK6812MINI_PLCC4_3.5x3.5mm_P1.75mm, F.Cu at (215.0, 124.1)
- added D306: SK6812MINI, LED_SMD:LED_SK6812MINI_PLCC4_3.5x3.5mm_P1.75mm, F.Cu at (215.0, 93.7)
- added D307: SK6812MINI, LED_SMD:LED_SK6812MINI_PLCC4_3.5x3.5mm_P1.75mm, F.Cu at (215.0, 63.4)
- added D308: SK6812MINI, LED_SMD:LED_SK6812MINI_PLCC4_3.5x3.5mm_P1.75mm, F.Cu at (202.6, 124.1)
- added D309: SK6812MINI, LED_SMD:LED_SK6812MINI_PLCC4_3.5x3.5mm_P1.75mm, F.Cu at (202.6, 93.7)
- added D310: SK6812MINI, LED_SMD:LED_SK6812MINI_PLCC4_3.5x3.5mm_P1.75mm, F.Cu at (202.6, 63.4)
- added D311: SK6812MINI, LED_SMD:LED_SK6812MINI_PLCC4_3.5x3.5mm_P1.75mm, F.Cu at (193.9, 115.4)
- added D312: SK6812MINI, LED_SMD:LED_SK6812MINI_PLCC4_3.5x3.5mm_P1.75mm, F.Cu at (193.9, 103.0)
- added D313: SK6812MINI, LED_SMD:LED_SK6812MINI_PLCC4_3.5x3.5mm_P1.75mm, F.Cu at (193.9, 84.5)
- added D314: SK6812MINI, LED_SMD:LED_SK6812MINI_PLCC4_3.5x3.5mm_P1.75mm, F.Cu at (193.9, 72.0)
- added D4: SK6812MINI, LED_SMD:LED_SK6812MINI_PLCC4_3.5x3.5mm_P1.75mm, F.Cu at (170.8, 101.6)
- added D401: SK6812MINI, LED_SMD:LED_SK6812MINI_PLCC4_3.5x3.5mm_P1.75mm, F.Cu at (118.0, 72.0)
- added D402: SK6812MINI, LED_SMD:LED_SK6812MINI_PLCC4_3.5x3.5mm_P1.75mm, F.Cu at (118.0, 84.5)
- added D403: SK6812MINI, LED_SMD:LED_SK6812MINI_PLCC4_3.5x3.5mm_P1.75mm, F.Cu at (118.0, 103.0)
- added D404: SK6812MINI, LED_SMD:LED_SK6812MINI_PLCC4_3.5x3.5mm_P1.75mm, F.Cu at (118.0, 115.4)
- added D405: SK6812MINI, LED_SMD:LED_SK6812MINI_PLCC4_3.5x3.5mm_P1.75mm, F.Cu at (126.6, 63.4)
- added D406: SK6812MINI, LED_SMD:LED_SK6812MINI_PLCC4_3.5x3.5mm_P1.75mm, F.Cu at (126.6, 93.7)
- added D407: SK6812MINI, LED_SMD:LED_SK6812MINI_PLCC4_3.5x3.5mm_P1.75mm, F.Cu at (126.6, 124.1)
- added D408: SK6812MINI, LED_SMD:LED_SK6812MINI_PLCC4_3.5x3.5mm_P1.75mm, F.Cu at (139.1, 63.4)
- added D409: SK6812MINI, LED_SMD:LED_SK6812MINI_PLCC4_3.5x3.5mm_P1.75mm, F.Cu at (139.1, 93.7)
- added D410: SK6812MINI, LED_SMD:LED_SK6812MINI_PLCC4_3.5x3.5mm_P1.75mm, F.Cu at (139.1, 124.1)
- added D411: SK6812MINI, LED_SMD:LED_SK6812MINI_PLCC4_3.5x3.5mm_P1.75mm, F.Cu at (147.7, 72.0)
- added D412: SK6812MINI, LED_SMD:LED_SK6812MINI_PLCC4_3.5x3.5mm_P1.75mm, F.Cu at (147.7, 84.5)
- added D413: SK6812MINI, LED_SMD:LED_SK6812MINI_PLCC4_3.5x3.5mm_P1.75mm, F.Cu at (147.7, 103.0)
- added D414: SK6812MINI, LED_SMD:LED_SK6812MINI_PLCC4_3.5x3.5mm_P1.75mm, F.Cu at (147.7, 115.4)
- added D5: SK6812MINI, LED_SMD:LED_SK6812MINI_PLCC4_3.5x3.5mm_P1.75mm, F.Cu at (170.8, 111.1)
- added D501: SK6812MINI, LED_SMD:LED_SK6812MINI_PLCC4_3.5x3.5mm_P1.75mm, F.Cu at (70.5, 72.0)
- added D502: SK6812MINI, LED_SMD:LED_SK6812MINI_PLCC4_3.5x3.5mm_P1.75mm, F.Cu at (70.5, 84.5)
- added D503: SK6812MINI, LED_SMD:LED_SK6812MINI_PLCC4_3.5x3.5mm_P1.75mm, F.Cu at (70.5, 103.0)
- added D504: SK6812MINI, LED_SMD:LED_SK6812MINI_PLCC4_3.5x3.5mm_P1.75mm, F.Cu at (70.5, 115.5)
- added D505: SK6812MINI, LED_SMD:LED_SK6812MINI_PLCC4_3.5x3.5mm_P1.75mm, F.Cu at (79.1, 63.4)
- added D506: SK6812MINI, LED_SMD:LED_SK6812MINI_PLCC4_3.5x3.5mm_P1.75mm, F.Cu at (79.1, 93.8)
- added D507: SK6812MINI, LED_SMD:LED_SK6812MINI_PLCC4_3.5x3.5mm_P1.75mm, F.Cu at (79.1, 124.1)
- added D508: SK6812MINI, LED_SMD:LED_SK6812MINI_PLCC4_3.5x3.5mm_P1.75mm, F.Cu at (91.6, 63.4)
- added D509: SK6812MINI, LED_SMD:LED_SK6812MINI_PLCC4_3.5x3.5mm_P1.75mm, F.Cu at (91.6, 93.8)
- added D510: SK6812MINI, LED_SMD:LED_SK6812MINI_PLCC4_3.5x3.5mm_P1.75mm, F.Cu at (91.6, 124.1)
- added D511: SK6812MINI, LED_SMD:LED_SK6812MINI_PLCC4_3.5x3.5mm_P1.75mm, F.Cu at (100.2, 72.0)
- added D512: SK6812MINI, LED_SMD:LED_SK6812MINI_PLCC4_3.5x3.5mm_P1.75mm, F.Cu at (100.2, 84.5)
- added D513: SK6812MINI, LED_SMD:LED_SK6812MINI_PLCC4_3.5x3.5mm_P1.75mm, F.Cu at (100.2, 103.0)
- added D514: SK6812MINI, LED_SMD:LED_SK6812MINI_PLCC4_3.5x3.5mm_P1.75mm, F.Cu at (100.2, 115.5)
- added D6: D_Schottky, Diode_SMD:D_TUMD2, F.Cu at (166.9, 93.2)
- added D7: D, Diode_SMD:D_SOD-123, F.Cu at (166.4, 91.1)
- added J1: USB_C_Receptacle_USB2.0, Connector_USB:USB_C_Receptacle_G-Switch_GT-USB-7010ASV, F.Cu at (170.8, 120.4)
- added J2: Barrel_Jack_Switch, Lib:1.3mmDCjack, B.Cu at (177.8, 90.8)
- added LS101: Speaker, Buzzer_Beeper:Buzzer_TDK_PS1240P02BT_D12.2mm_H6.5mm, B.Cu at (181.2, 104.8)
- added Q1: Q_Photo_NPN_CE, LED_THT:LED_D1.8mm_W1.8mm_H2.4mm_Horizontal_O3.81mm_Z1.6mm, F.Cu at (110.2, 76.5)
- added Q2: PMOS, Package_TO_SOT_SMD:SOT-23, F.Cu at (160.4, 88.4)
- added Q3: PMOS, Package_TO_SOT_SMD:SOT-23, F.Cu at (160.4, 92.7)
- added R1: 5.1k, Resistor_SMD:R_0603_1608Metric_Pad0.98x0.95mm_HandSolder, F.Cu at (176.9, 122.6)
- added R2: 5.1k, Resistor_SMD:R_0603_1608Metric_Pad0.98x0.95mm_HandSolder, F.Cu at (164.6, 122.6)
- added R3: 100k, Resistor_SMD:R_0603_1608Metric_Pad0.98x0.95mm_HandSolder, F.Cu at (109.0, 88.3)
- added R4: 10k, Resistor_SMD:R_0603_1608Metric_Pad0.98x0.95mm_HandSolder, F.Cu at (163.2, 90.0)
- added R5: 10k, Resistor_SMD:R_0603_1608Metric_Pad0.98x0.95mm_HandSolder, F.Cu at (180.2, 87.6)
- added R6: 10k, Resistor_SMD:R_0603_1608Metric_Pad0.98x0.95mm_HandSolder, F.Cu at (180.2, 86.1)
- added REF**: StampHole, Lib:StampHole, F.Cu at (166.5, 116.6)
- added SW1: EN, Button_Switch_SMD:SW_Push_1P1T_NO_Vertical_Wuerth_434133025816, F.Cu at (160.7, 109.3)
- added SW2: BOOT, Button_Switch_SMD:SW_Push_1P1T_NO_Vertical_Wuerth_434133025816, F.Cu at (160.7, 104.8)
- added U1: ESP32-C3-WROOM-02, Espressif:ESP32-C3-WROOM-02, B.Cu at (175.6, 80.5)
- added U2: LM1117GS-3.3, Package_TO_SOT_SMD:SOT-223, F.Cu at (184.2, 96.4)
Routing:
- net +5V: track 0.00 -> 1032.4 mm
- net /Sheetname: 7-Segment-ARGB3/DIN: track 0.00 -> 98.6 mm, vias 0 -> 1
- net LS: track 0.00 -> 97.6 mm, vias 0 -> 3
- net /Sheetname: 7-Segment-ARGB/DIN: track 0.00 -> 79.9 mm, vias 0 -> 1
- net /Sheetname: 7-Segment-ARGB2/DIN: track 0.00 -> 47.0 mm, vias 0 -> 1
- net SPEAK: track 0.00 -> 43.8 mm, vias 0 -> 1
- net D+: track 0.00 -> 37.9 mm, vias 0 -> 1
- net D-: track 0.00 -> 37.2 mm, vias 0 -> 1
- net Net-(U1-EN/CHIP_PU): track 0.00 -> 34.8 mm, vias 0 -> 3
- net Net-(D1-DOUT): track 0.00 -> 33.0 mm, vias 0 -> 2
- net /Sheetname: 7-Segment-ARGB1/DIN: track 0.00 -> 31.3 mm, vias 0 -> 1
- net Net-(D509-DOUT): track 0.00 -> 29.2 mm
- net Net-(D309-DOUT): track 0.00 -> 29.2 mm
- net Net-(D209-DOUT): track 0.00 -> 29.2 mm
- net Net-(D409-DOUT): track 0.00 -> 29.2 mm
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- added copper zone on B.Cu, net D+
- added copper zone on F.Cu, net D+
- added copper zone on B.Cu, net D-
- added copper zone on F.Cu, net D-
- added copper zone on B.Cu, net GND
- added copper zone on F.Cu, net GND
- added copper zone on B.Cu, net USB5V
- added copper zone on F.Cu, net USB5V
Other:
- outline, holes or cut-outs redrawn

Commit message: pcb
Parts:
- removed Q2, Q3: PMOS, Package_TO_SOT_SMD:SOT-23
- removed R4: 10k, Resistor_SMD:R_0603_1608Metric_Pad0.98x0.95mm_HandSolder
- removed REF**: StampHole, Lib:StampHole
- D7: value D -> D_Schottky; footprint Diode_SMD:D_SOD-123 -> Diode_SMD:D_TUMD2
- J1: value USB_C_Receptacle_USB2.0 -> USB4145-03-0230-C; footprint Connector_USB:USB_C_Receptacle_G-Switch_GT-USB-7010ASV -> Lib:USB4145030230C; moved to B.Cu
- R1, R2: moved to B.Cu
- moved R1 35.5 mm to (159.5, 91.6), turned to 90 degrees
- moved J1 26.7 mm to (158.4, 96.8)
- moved R2 22.6 mm to (157.5, 101.1), turned to 180 degrees
- moved D6 3.31 mm to (169.7, 91.4)
- moved C202 2.01 mm to (272.5, 110.5), turned to -90 degrees
- moved C505 2.00 mm to (86.6, 62.0), turned to 0 degrees
- moved C502 2.00 mm to (69.1, 77.0), turned to 90 degrees
- moved C305 1.99 mm to (207.5, 125.5), turned to 180 degrees
- moved C402 1.98 mm to (116.6, 77.0), turned to 90 degrees
- moved C405 1.98 mm to (134.1, 62.0), turned to 0 degrees
- moved C205 1.98 mm to (255.0, 125.5), turned to 180 degrees
- moved C302 1.97 mm to (225.0, 110.5), turned to -90 degrees
- moved C307 1.84 mm to (192.5, 108.0), turned to 90 degrees
- moved C407 1.83 mm to (149.1, 79.5), turned to -90 degrees
- moved C507 1.82 mm to (101.6, 79.5), turned to -90 degrees
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- renumbered D2 to D1, D1 to D2
Connections:
- D2 pad 1: Net-(D1-DOUT) (its old number) -> Net-(D2-DOUT)
- D201 pad 1: unconnected-(D201-DOUT-Pad1) -> Net-(D201-DOUT)
- D202 pad 3: Net-(D201-DIN) -> Net-(D201-DOUT)
- D204 pad 1: unconnected-(D204-DOUT-Pad1) -> Net-(D203-DIN)
- D204 pad 3: Net-(D203-DIN) -> Net-(D204-DIN)
- D206 pad 1: unconnected-(D206-DOUT-Pad1) -> Net-(D206-DOUT)
- D207 pad 1: Net-(D203-DIN) -> Net-(D204-DIN)
- D208 pad 1: unconnected-(D208-DOUT-Pad1) -> Net-(D205-DIN)
- D208 pad 3: Net-(D205-DIN) -> Net-(D208-DIN)
- D209 pad 3: Net-(D203-DOUT) -> Net-(D206-DOUT)
- D210 pad 1: unconnected-(D210-DOUT-Pad1) -> Net-(D207-DIN)
- D210 pad 3: Net-(D207-DIN) -> Net-(D210-DIN)
- D211 pad 1: Net-(D205-DIN) -> Net-(D208-DIN)
- D211 pad 3: Net-(D209-DOUT) -> Net-(D211-DIN)
- D212 pad 1: unconnected-(D212-DOUT-Pad1) -> Net-(D211-DIN)
- D213 pad 1: unconnected-(D213-DOUT-Pad1) -> Net-(D213-DOUT)
- D213 pad 3: /Sheetname: 7-Segment-ARGB/DIN -> /Sheetname: 7-Segment-ARGB2/DIN
- D214 pad 1: Net-(D207-DIN) -> Net-(D210-DIN)
- D214 pad 3: /Sheetname: 7-Segment-ARGB/DIN -> Net-(D213-DOUT)
- D3 pad 1: unconnected-(D3-DOUT-Pad1) -> Net-(D3-DOUT)
- D3 pad 3: Net-(D1-DOUT) (its old number) -> Net-(D2-DOUT)
- D301 pad 1: unconnected-(D301-DOUT-Pad1) -> Net-(D301-DOUT)
- D302 pad 3: Net-(D301-DIN) -> Net-(D301-DOUT)
- D304 pad 1: unconnected-(D304-DOUT-Pad1) -> Net-(D303-DIN)
- D304 pad 3: Net-(D303-DIN) -> Net-(D304-DIN)
- D306 pad 1: unconnected-(D306-DOUT-Pad1) -> Net-(D306-DOUT)
- D307 pad 1: Net-(D303-DIN) -> Net-(D304-DIN)
- D308 pad 1: unconnected-(D308-DOUT-Pad1) -> Net-(D305-DIN)
- D308 pad 3: Net-(D305-DIN) -> Net-(D308-DIN)
- D309 pad 3: Net-(D303-DOUT) -> Net-(D306-DOUT)
- D310 pad 1: unconnected-(D310-DOUT-Pad1) -> Net-(D307-DIN)
- D310 pad 3: Net-(D307-DIN) -> Net-(D310-DIN)
- D311 pad 1: Net-(D305-DIN) -> Net-(D308-DIN)
- D311 pad 3: Net-(D309-DOUT) -> Net-(D311-DIN)
- D312 pad 1: unconnected-(D312-DOUT-Pad1) -> Net-(D311-DIN)
- D313 pad 1: unconnected-(D313-DOUT-Pad1) -> Net-(D313-DOUT)
- D314 pad 1: Net-(D307-DIN) -> Net-(D310-DIN)
- D314 pad 3: /Sheetname: 7-Segment-ARGB1/DIN -> Net-(D313-DOUT)
- D4 pad 3: Net-(D1-DOUT) (its old number) -> Net-(D3-DOUT)
- D401 pad 1: unconnected-(D401-DOUT-Pad1) -> Net-(D401-DOUT)
- D402 pad 3: Net-(D401-DIN) -> Net-(D401-DOUT)
- D404 pad 1: unconnected-(D404-DOUT-Pad1) -> Net-(D403-DIN)
- D404 pad 3: Net-(D403-DIN) -> Net-(D404-DIN)
- D406 pad 1: unconnected-(D406-DOUT-Pad1) -> Net-(D406-DOUT)
- D407 pad 1: Net-(D403-DIN) -> Net-(D404-DIN)
- D408 pad 1: unconnected-(D408-DOUT-Pad1) -> Net-(D405-DIN)
- D408 pad 3: Net-(D405-DIN) -> Net-(D408-DIN)
- D409 pad 3: Net-(D403-DOUT) -> Net-(D406-DOUT)
- D410 pad 1: unconnected-(D410-DOUT-Pad1) -> Net-(D407-DIN)
- D410 pad 3: Net-(D407-DIN) -> Net-(D410-DIN)
- D411 pad 1: Net-(D405-DIN) -> Net-(D408-DIN)
- D411 pad 3: Net-(D409-DOUT) -> Net-(D411-DIN)
- D412 pad 1: unconnected-(D412-DOUT-Pad1) -> Net-(D411-DIN)
- D413 pad 1: unconnected-(D413-DOUT-Pad1) -> Net-(D413-DOUT)
- D413 pad 3: /Sheetname: 7-Segment-ARGB2/DIN -> /Sheetname: 7-Segment-ARGB3/DIN
- D414 pad 1: Net-(D407-DIN) -> Net-(D410-DIN)
- D414 pad 3: /Sheetname: 7-Segment-ARGB2/DIN -> Net-(D413-DOUT)
- D501 pad 1: unconnected-(D501-DOUT-Pad1) -> Net-(D501-DOUT)
- D502 pad 3: Net-(D501-DIN) -> Net-(D501-DOUT)
- D504 pad 1: unconnected-(D504-DOUT-Pad1) -> Net-(D503-DIN)
- D504 pad 3: Net-(D503-DIN) -> Net-(D504-DIN)
- D506 pad 1: unconnected-(D506-DOUT-Pad1) -> Net-(D506-DOUT)
- D507 pad 1: Net-(D503-DIN) -> Net-(D504-DIN)
- D508 pad 1: unconnected-(D508-DOUT-Pad1) -> Net-(D505-DIN)
- D508 pad 3: Net-(D505-DIN) -> Net-(D508-DIN)
- D509 pad 3: Net-(D503-DOUT) -> Net-(D506-DOUT)
- D510 pad 1: unconnected-(D510-DOUT-Pad1) -> Net-(D507-DIN)
- D510 pad 3: Net-(D507-DIN) -> Net-(D510-DIN)
- D511 pad 1: Net-(D505-DIN) -> Net-(D508-DIN)
- D511 pad 3: Net-(D509-DOUT) -> Net-(D511-DIN)
- D512 pad 1: unconnected-(D512-DOUT-Pad1) -> Net-(D511-DIN)
- D513 pad 1: unconnected-(D513-DOUT-Pad1) -> Net-(D513-DOUT)
- D513 pad 3: /Sheetname: 7-Segment-ARGB3/DIN -> /Sheetname: 7-Segment-ARGB4/DIN
- D514 pad 1: Net-(D507-DIN) -> Net-(D510-DIN)
- D514 pad 3: /Sheetname: 7-Segment-ARGB3/DIN -> Net-(D513-DOUT)
- D7 pad 1: Net-(D7-K) -> +5V
- D7 pad 2: DC5V -> USB5V
- U1 pad 4: /Sheetname: 7-Segment-ARGB/DIN -> /Sheetname: 7-Segment-ARGB2/DIN
- U1 pad 5: /Sheetname: 7-Segment-ARGB2/DIN -> /Sheetname: 7-Segment-ARGB4/DIN
Routing:
- net /Sheetname: 7-Segment-ARGB4/DIN: track 0.00 -> 85.2 mm, vias 0 -> 1
- net /Sheetname: 7-Segment-ARGB/DIN: track 79.9 -> 0.00 mm, vias 1 -> 0
- net +5V: track 1032.4 -> 958.6 mm
- net /Sheetname: 7-Segment-ARGB3/DIN: track 98.6 -> 32.7 mm
- net Net-(D1-DOUT) (its old number): track 33.0 -> 0.00 mm, vias 2 -> 0
- net Net-(D3-DOUT): track 0.00 -> 20.5 mm, vias 0 -> 2
- net /Sheetname: 7-Segment-ARGB2/DIN: track 47.0 -> 66.6 mm
- net Net-(D203-DIN): track 28.1 -> 9.67 mm
- net Net-(D507-DIN): track 28.1 -> 9.67 mm
- net Net-(D503-DIN): track 28.1 -> 9.67 mm
- net Net-(D407-DIN): track 28.1 -> 9.67 mm
- net Net-(D403-DIN): track 28.1 -> 9.67 mm
- net Net-(D307-DIN): track 28.1 -> 9.67 mm
- net Net-(D207-DIN): track 28.1 -> 9.67 mm
- net Net-(D303-DIN): track 28.1 -> 9.67 mm
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- removed copper zone on B.Cu, net D+
- removed copper zone on F.Cu, net D+
- removed copper zone on B.Cu, net D-
- removed copper zone on F.Cu, net D-
- removed copper zone on B.Cu, net USB5V
- removed copper zone on F.Cu, net USB5V
Other:
- outline, holes or cut-outs redrawn
