File: gaming-clock/untitled.kicad_sch (KiCad schematic)
At the start: 14 parts

Commit message: c
Parts:
- added C4 (x7): 10u, Capacitor_SMD:C_0603_1608Metric_Pad1.08x0.95mm_HandSolder, symbol Device:C
Connections:
- net +5V: now also C4.1, C4.1, C4.1, C4.1, C4.1, C4.1, C4.1
- net GND: now also C4.2, C4.2, C4.2, C4.2, C4.2, C4.2, C4.2

Commit message: fin
Connections:
- net GND: now also D10.2 (VSS), D11.2 (VSS)

Commit message: pcb
Connections:
- net DIN: no longer D13.3 (DIN)
- net at D3.1 (DOUT): now also D2.3 (DIN)
- net at D3.3 (DIN), D4.1 (DOUT): no longer D2.3 (DIN)
- net at D2.1 (DOUT), D6.3 (DIN): no longer D7.3 (DIN)
- net at D14.1 (DOUT): now also D15.3 (DIN)
- net at D13.1 (DOUT), D14.3 (DIN): no longer D15.3 (DIN)
- net at D15.1 (DOUT), D9.3 (DIN): no longer D8.3 (DIN)
- net at D9.1 (DOUT): now also D8.3 (DIN)
- net at D6.1 (DOUT): now also D7.3 (DIN)
- net at D12.1 (DOUT): now also D13.3 (DIN)
- net at D10.1 (DOUT): now also D11.3 (DIN)
- net at D10.3 (DIN), D8.1 (DOUT): no longer D11.3 (DIN)
- net at D5.1 (DOUT): now also D4.3 (DIN)
- net at D11.1 (DOUT), D5.3 (DIN): no longer D4.3 (DIN)
